Commit message: Göruntu Birleşştirme

File: description/camera6.xacro (robot description, xacro)
@@ -1,10 +1,10 @@
 <?xml version="1.0"?>
 <robot xmlns:xacro="http://www.ros.org/wiki/xacro" >
-    <joint name="camera_joint" type="fixed">
+    <joint name="camera_6_joint" type="fixed">
         <parent link="chassis"/>
-        <child link="camera_link"/>
-        <origin xyz="0.305 0 0.08" rpy="0 0 0"/>
+        <child link="camera_6_link"/>
+        <origin xyz="0.305  0 0.25" rpy="0 0 ${-5*pi/3}"/>
     </joint>
-    <link name="camera_link">
+    <link name="camera_6_link">
         <visual>
             <geometry>
@@ -14,18 +14,19 @@
         </visual>
     </link>
-    <joint name="camera_optical_joint" type="fixed">
-        <parent link="camera_link"/>
-        <child link="camera_link_optical"/>
+    <joint name="camera_6_optical_joint" type="fixed">
+        <parent link="camera_6_link"/>
+        <child link="camera_6_link_optical"/>
         <origin xyz="0 0 0" rpy="${-pi/2} 0 ${-pi/2}"/>
     </joint>
-    <link name="camera_link_optical"></link>
-    <gazebo reference="camera_link">
+    <link name="camera_6_link_optical"></link>
+    <gazebo reference="camera_6_link">
         <material>Gazebo/Red</material>
-        <sensor name="camera" type="camera">
+        <sensor name="camera_6" type="camera">
             <pose> 0 0 0 0 0 0 </pose>
             <visualize>true</visualize>
             <update_rate>10</update_rate>
             <camera>
-                <horizontal_fov>1.089</horizontal_fov>
+                <horizontal_fov>2.094</horizontal_fov>
+                <vertical_fov>2.094</vertical_fov>
                 <image>
                     <format>R8G8B8</format>
@@ -38,6 +39,6 @@
                 </clip>
             </camera>
-            <plugin name="camera_controller" filename="libgazebo_ros_camera.so">
-                <frame_name>camera_link_optical</frame_name>
+            <plugin name="camera_6_controller" filename="libgazebo_ros_camera.so">
+                <frame_name>camera_6_link_optical</frame_name>
             </plugin>
         </sensor>

File: description/robot.urdf.xacro (robot description, xacro)
@@ -3,6 +3,11 @@
     <xacro:include filename="robot_core.xacro" />
     <xacro:include filename="gazebo_control.xacro" />
-    <xacro:include filename="lidar.xacro" />
-    <!--xacro:include filename="camera.xacro" />-->
-    <xacro:include filename="depth_camera.xacro" />
+    <!--<xacro:include filename="lidar.xacro" />-->
+    <xacro:include filename="camera1.xacro" />
+    <xacro:include filename="camera2.xacro" />
+    <xacro:include filename="camera3.xacro" />
+    <xacro:include filename="camera4.xacro" />
+    <xacro:include filename="camera5.xacro" />
+    <xacro:include filename="camera6.xacro" />
+    <!--<xacro:include filename="depth_camera.xacro" />-->
 </robot>
