Commit message: Robot Sürekli Kamera Dödnürme

File: description/camera1.xacro (robot description, xacro)
@@ -1,10 +1,34 @@
 <?xml version="1.0"?>
-<robot xmlns:xacro="http://www.ros.org/wiki/xacro" >
-    <joint name="camera_1_joint" type="fixed">
+<robot xmlns:xacro="http://www.ros.org/wiki/xacro">
+    <joint name="camera_1_joint" type="revolute">
+        <!-- Parent ve child linkleri belirtin -->
         <parent link="chassis"/>
         <child link="camera_1_link"/>
-        <origin xyz="0.305 0 0.25" rpy="0 0 0 "/>
+        <!-- Origin ve axis değerlerini belirtin -->
+        <origin xyz="0.305 0 0.25" rpy="0 0 0"/>
+        <axis xyz="0 0 1"/>
+        <!-- Joint limitlerini belirtin -->
+        <limit effort="1000" lower="-3.14" upper="3.14" velocity="1.57"/>
     </joint>
+    <gazebo>
+        <plugin name="gazebo_ros_joint_state_publisher"
+            filename="libgazebo_ros_joint_state_publisher.so">
+            <update_rate>20</update_rate>
+            <joint_name>camera_1_joint</joint_name>
+        </plugin>
+    </gazebo>
+    <gazebo>
+        <plugin name="gazebo_ros_joint_pose_trajectory"
+            filename="libgazebo_ros_joint_pose_trajectory.so">
+            <update_rate>2</update_rate>
+            <joint_name>camera_1_joint</joint_name>
+        </plugin>
+    </gazebo>
     <link name="camera_1_link">
+        <inertial>
+            <origin xyz="0 0 0" rpy="0 0 0"/>
+            <mass value="1"/>
+            <inertia ixx="1" ixy="0" ixz="0" iyy="1" iyz="0" izz="1"/>
+        </inertial>
         <visual>
             <geometry>

File: description/robot.urdf.xacro (robot description, xacro)
@@ -6,8 +6,8 @@
     <xacro:include filename="camera1.xacro" />
     <xacro:include filename="camera2.xacro" />
-    <xacro:include filename="camera3.xacro" />
+    <!--<xacro:include filename="camera3.xacro" />
     <xacro:include filename="camera4.xacro" />
     <xacro:include filename="camera5.xacro" />
-    <xacro:include filename="camera6.xacro" />
+    <xacro:include filename="camera6.xacro" />-->
     <!--<xacro:include filename="depth_camera.xacro" />-->
 </robot>
